Commit message: Added gazebo launch files for robotiq gripper

File: robotiq_s_model_visualization/cfg/s-model_articulated.xacro (robot description, xacro)
@@ -8,5 +8,5 @@
 	<xacro:s-model_articulated prefix=""/>
 <!--
-	<xacro:include filename="$(find robotiq_s_model_visualization)/cfg/s-model_finger_articulated_macro.xacro" />
+	<include filename="$(find robotiq_s_model_visualization)/cfg/s-model_finger_articulated_macro.xacro" />
 	<xacro:s-model_finger_articulated prefix=""/>
 -->

File: robotiq_s_model_visualization/cfg/s-model_articulated_macro.xacro (robot description, xacro)
@@ -7,9 +7,12 @@
 <robot xmlns:xacro="http://ros.org/wiki/xacro">
 	<xacro:include filename="$(find robotiq_s_model_visualization)/cfg/s-model_finger_articulated_macro.xacro" />
-	<xacro:macro name="s-model_articulated" params="prefix parent *origin">
+	<xacro:macro name="s-model_articulated" params="prefix">
 	<xacro:s-model_finger_articulated prefix="${prefix}finger_1_"/>
 	<xacro:s-model_finger_articulated prefix="${prefix}finger_2_"/>
 	<xacro:s-model_finger_articulated prefix="${prefix}finger_middle_"/>
-		<!-- link list -->
+        <!-- Gazebo plugin for ROS Control -->
+        <!-- <gazebo>
+            <plugin name="ros_control" filename="libgazebo_ros_control.so"/> -->
+                <!-- link list -->
 		<link name="${prefix}palm">
 			<visual>
@@ -37,10 +40,4 @@
 		<!-- end of link list -->
 		<!-- joint list -->
-    <!-- Joint to conect with robot parent-->
-    <joint name="${prefix}robotiq_hand_joint" type="fixed">
-      <insert_block name="origin"/>
-      <parent link="${parent}"/>
-      <child link="${prefix}palm"/>
-    </joint>
 		<!-- WARNING: LIMITS NOT CORRECT -->
 		<joint name="${prefix}palm_finger_1_joint" type="revolute">
