Commit message: [robotiq-s_model_visualization] * Added parameters to xacro file to consider a parent robot

File: robotiq_s_model_visualization/cfg/s-model_articulated_macro.xacro (robot description, xacro)
@@ -7,5 +7,5 @@
 <robot xmlns:xacro="http://ros.org/wiki/xacro">
 	<xacro:include filename="$(find robotiq_s_model_visualization)/cfg/s-model_finger_articulated_macro.xacro" />
-	<xacro:macro name="s-model_articulated" params="prefix">
+	<xacro:macro name="s-model_articulated" params="prefix parent *origin">
 	<xacro:s-model_finger_articulated prefix="${prefix}finger_1_"/>
 	<xacro:s-model_finger_articulated prefix="${prefix}finger_2_"/>
@@ -37,4 +37,10 @@
 		<!-- end of link list -->
 		<!-- joint list -->
+    <!-- Joint to conect with robot parent-->
+    <joint name="${prefix}robotiq_hand_joint" type="fixed">
+      <insert_block name="origin"/>
+      <parent link="${parent}"/>
+      <child link="${prefix}palm"/>
+    </joint>
 		<!-- WARNING: LIMITS NOT CORRECT -->
 		<joint name="${prefix}palm_finger_1_joint" type="revolute">

Commit message: Added black colors over the white null mesh

File: robotiq_s_model_visualization/cfg/s-model_articulated_macro.xacro (robot description, xacro)
@@ -20,7 +20,4 @@
 					<mesh filename="package://robotiq_s_model_visualization/meshes/s-model_articulated/visual/palm.STL" />
 				</geometry>
-				<material name="green">
-					<color rgba="0 1 0 1"/>
-				</material>
 			</visual>
 			<collision>
@@ -28,9 +25,9 @@
 					<mesh filename="package://robotiq_s_model_visualization/meshes/s-model_articulated/collision/palm.STL" />
 				</geometry>
-				<material name="yellow">
-					<color rgba="0 1 1 1"/>
-				</material>
 			</collision>
 		</link>
+                <gazebo reference="${prefix}palm">
+                    <material>Gazebo/Black</material>
+                </gazebo>
         <inertial>
             <origin xyz="0 0 0" rpy="0 0 0"/>

File: robotiq_s_model_visualization/cfg/s-model_finger_articulated_macro.xacro (robot description, xacro)
@@ -14,7 +14,4 @@
 					<mesh filename="package://robotiq_s_model_visualization/meshes/s-model_articulated/visual/link_0.STL" />
 				</geometry>
-				<material name="green">
-					<color rgba="0 1 0 1"/>
-				</material>
 			</visual>
 			<collision>
@@ -23,7 +20,4 @@
 					<mesh filename="package://robotiq_s_model_visualization/meshes/s-model_articulated/collision/link_0.STL" />
 				</geometry>
-				<material name="yellow">
-					<color rgba="0 1 1 1"/>
-				</material>
 			</collision>
             <inertial>
@@ -33,4 +27,7 @@
             </inertial>
 		</link>
+  <gazebo reference="${prefix}link_0">
+                            <material>Gazebo/Black</material>
+                        </gazebo>
 		<link name="${prefix}link_1">
 			<visual>
@@ -39,5 +36,4 @@
 					<mesh filename="package://robotiq_s_model_visualization/meshes/s-model_articulated/visual/link_1.STL" />
 				</geometry>
-				<material name="green"/>
 			</visual>
 			<collision>
@@ -46,5 +42,4 @@
 					<mesh filename="package://robotiq_s_model_visualization/meshes/s-model_articulated/collision/link_1.STL" />
 				</geometry>
-				<material name="yellow"/>
 			</collision>
             <inertial>
@@ -54,4 +49,7 @@
             </inertial>
 		</link>
+ <gazebo reference="${prefix}link_1">
+                            <material>Gazebo/Black</material>
+                        </gazebo>
 		<link name="${prefix}link_2">
 			<!--
@@ -65,5 +63,4 @@
 					<mesh filename="package://robotiq_s_model_visualization/meshes/s-model_articulated/visual/link_2.STL" />
 				</geometry>
-				<material name="green"/>
 			</visual>
 			<collision>
@@ -72,5 +69,4 @@
 					<mesh filename="package://robotiq_s_model_visualization/meshes/s-model_articulated/collision/link_2.STL" />
 				</geometry>
-				<material name="yellow"/>
 			</collision>
             <inertial>
@@ -80,4 +76,7 @@
             </inertial>
 		</link>
+ <gazebo reference="${prefix}link_2">
+				<material>Gazebo/Black</material>
+                                </gazebo>
 		<link name="${prefix}link_3">
 			<visual>
@@ -86,5 +85,4 @@
 					<mesh filename="package://robotiq_s_model_visualization/meshes/s-model_articulated/visual/link_3.STL" />
 				</geometry>
-				<material name="green"/>
 			</visual>
 			<collision>
@@ -93,5 +91,4 @@
 					<mesh filename="package://robotiq_s_model_visualization/meshes/s-model_articulated/collision/link_3.STL" />
 				</geometry>
-				<material name="yellow"/>
 			</collision>
             <inertial>
@@ -101,4 +98,7 @@
             </inertial>
 		</link>
+<gazebo reference="${prefix}link_2">
+				<material>Gazebo/Black</material>
+                                </gazebo>
 		<!-- end of link list -->
 		<!-- joint list -->

Commit message: Added self collides on robotiq model

File: robotiq_s_model_visualization/cfg/s-model_articulated_macro.xacro (robot description, xacro)
@@ -27,7 +27,7 @@
 			</collision>
 		</link>
-                <gazebo reference="${prefix}palm">
-                    <material>Gazebo/Black</material>
-                </gazebo>
+        <gazebo reference="${prefix}palm">
+            <selfCollide>true</selfCollide>
+        </gazebo>
         <inertial>
             <origin xyz="0 0 0" rpy="0 0 0"/>

File: robotiq_s_model_visualization/cfg/s-model_finger_articulated_macro.xacro (robot description, xacro)
@@ -27,7 +27,8 @@
             </inertial>
 		</link>
-  <gazebo reference="${prefix}link_0">
-                            <material>Gazebo/Black</material>
-                        </gazebo>
+                <gazebo reference="${prefix}link_0">
+                    <material>Gazebo/Black</material>
+                    <selfCollide>true</selfCollide>
+                </gazebo>
 		<link name="${prefix}link_1">
 			<visual>
@@ -49,7 +50,8 @@
             </inertial>
 		</link>
- <gazebo reference="${prefix}link_1">
+                 <gazebo reference="${prefix}link_1">
                             <material>Gazebo/Black</material>
-                        </gazebo>
+                            <selfCollide>true</selfCollide>
+                 </gazebo>
 		<link name="${prefix}link_2">
 			<!--
@@ -78,4 +80,5 @@
  <gazebo reference="${prefix}link_2">
 				<material>Gazebo/Black</material>
+                                <selfCollide>true</selfCollide>
                                 </gazebo>
 		<link name="${prefix}link_3">
@@ -100,4 +103,5 @@
 <gazebo reference="${prefix}link_2">
 				<material>Gazebo/Black</material>
+                                <selfCollide>true</selfCollide>
                                 </gazebo>
 		<!-- end of link list -->

Commit message: Added things

File: robotiq_s_model_visualization/cfg/s-model_articulated_macro.xacro (robot description, xacro)
@@ -5,14 +5,15 @@
 there are multiple hands then a prefix followed by an "_" is needed.
 -->
+        <!-- Gazebo plugin for ROS Control -->
+        <!-- <gazebo>
+            <plugin name="ros_control" filename="libgazebo_ros_control.so"/>
+-->
 <robot xmlns:xacro="http://ros.org/wiki/xacro">
-	<xacro:include filename="$(find robotiq_s_model_visualization)/cfg/s-model_finger_articulated_macro.xacro" />
+	<!-- <xacro:include filename="$(find robotiq_s_model_visualization)/cfg/s-model_finger_articulated_macro.xacro" /> -->
 	<xacro:macro name="s-model_articulated" params="prefix">
-	<xacro:s-model_finger_articulated prefix="${prefix}finger_1_"/>
+	<!-- <xacro:s-model_finger_articulated prefix="${prefix}finger_1_"/>
 	<xacro:s-model_finger_articulated prefix="${prefix}finger_2_"/>
 	<xacro:s-model_finger_articulated prefix="${prefix}finger_middle_"/>
-        <!-- Gazebo plugin for ROS Control -->
-        <!-- <gazebo>
-            <plugin name="ros_control" filename="libgazebo_ros_control.so"/> -->
-                <!-- link list -->
+-->
 		<link name="${prefix}palm">
 			<visual>
@@ -27,7 +28,4 @@
 			</collision>
 		</link>
-        <gazebo reference="${prefix}palm">
-            <selfCollide>true</selfCollide>
-        </gazebo>
         <inertial>
             <origin xyz="0 0 0" rpy="0 0 0"/>
@@ -38,5 +36,5 @@
 		<!-- joint list -->
 		<!-- WARNING: LIMITS NOT CORRECT -->
-		<joint name="${prefix}palm_finger_1_joint" type="revolute">
+	<!--	<joint name="${prefix}palm_finger_1_joint" type="revolute">
 			<parent link="${prefix}palm"/>
 			<child link="${prefix}finger_1_link_0"/>
@@ -44,6 +42,4 @@
 			<origin xyz="-0.0455 0.0214 0.036" rpy="0 3.1416 -1.57"/>
 			<limit lower="-0.16" upper="0.25" effort="100" velocity="100"/>
-		</joint>
-		<!-- WARNING: LIMITS NOT CORRECT -->
 		<joint name="${prefix}palm_finger_2_joint" type="revolute">
 			<parent link="${prefix}palm"/>
@@ -58,6 +54,5 @@
 			<axis xyz="0 0 1"/>
 			<origin xyz="0.0455 0.0214 0" rpy="0 0 1.57"/>
-		</joint>
-		<!-- end of joint list -->
+		</joint> -->
 	</xacro:macro>
 </robot>

File: robotiq_s_model_visualization/cfg/s-model_finger_articulated_macro.xacro (robot description, xacro)
@@ -29,5 +29,5 @@
                 <gazebo reference="${prefix}link_0">
                     <material>Gazebo/Black</material>
-                    <selfCollide>true</selfCollide>
+                    <selfCollide>false</selfCollide>
                 </gazebo>
 		<link name="${prefix}link_1">
@@ -52,5 +52,5 @@
                  <gazebo reference="${prefix}link_1">
                             <material>Gazebo/Black</material>
-                            <selfCollide>true</selfCollide>
+                            <selfCollide>false</selfCollide>
                  </gazebo>
 		<link name="${prefix}link_2">
@@ -80,5 +80,5 @@
  <gazebo reference="${prefix}link_2">
 				<material>Gazebo/Black</material>
-                                <selfCollide>true</selfCollide>
+                                <selfCollide>false</selfCollide>
                                 </gazebo>
 		<link name="${prefix}link_3">
@@ -103,5 +103,5 @@
 <gazebo reference="${prefix}link_2">
 				<material>Gazebo/Black</material>
-                                <selfCollide>true</selfCollide>
+                                <selfCollide>false</selfCollide>
                                 </gazebo>
 		<!-- end of link list -->

Commit message: Fixed

File: robotiq_s_model_visualization/cfg/s-model_articulated_macro.xacro (robot description, xacro)
@@ -10,10 +10,9 @@
 -->
 <robot xmlns:xacro="http://ros.org/wiki/xacro">
-	<!-- <xacro:include filename="$(find robotiq_s_model_visualization)/cfg/s-model_finger_articulated_macro.xacro" /> -->
+	<xacro:include filename="$(find robotiq_s_model_visualization)/cfg/s-model_finger_articulated_macro.xacro" />
 	<xacro:macro name="s-model_articulated" params="prefix">
-	<!-- <xacro:s-model_finger_articulated prefix="${prefix}finger_1_"/>
+	<xacro:s-model_finger_articulated prefix="${prefix}finger_1_"/>
 	<xacro:s-model_finger_articulated prefix="${prefix}finger_2_"/>
 	<xacro:s-model_finger_articulated prefix="${prefix}finger_middle_"/>
--->
 		<link name="${prefix}palm">
 			<visual>
@@ -36,5 +35,5 @@
 		<!-- joint list -->
 		<!-- WARNING: LIMITS NOT CORRECT -->
-	<!--	<joint name="${prefix}palm_finger_1_joint" type="revolute">
+		<joint name="${prefix}palm_finger_1_joint" type="revolute">
 			<parent link="${prefix}palm"/>
 			<child link="${prefix}finger_1_link_0"/>
@@ -42,4 +41,5 @@
 			<origin xyz="-0.0455 0.0214 0.036" rpy="0 3.1416 -1.57"/>
 			<limit lower="-0.16" upper="0.25" effort="100" velocity="100"/>
+                </joint>
 		<joint name="${prefix}palm_finger_2_joint" type="revolute">
 			<parent link="${prefix}palm"/>
@@ -54,5 +54,5 @@
 			<axis xyz="0 0 1"/>
 			<origin xyz="0.0455 0.0214 0" rpy="0 0 1.57"/>
-		</joint> -->
+		</joint>
 	</xacro:macro>
 </robot>

Commit message: Removed broken gripper collision tag, prevented MoveIt use

File: robotiq_s_model_visualization/cfg/s-model_articulated_macro.xacro (robot description, xacro)
@@ -27,4 +27,7 @@
 			</collision>
 		</link>
+                <gazebo reference="${prefix}palm">
+                        <material>Gazebo/Blue</material>
+                </gazebo>
         <inertial>
             <origin xyz="0 0 0" rpy="0 0 0"/>

File: robotiq_s_model_visualization/cfg/s-model_finger_articulated_macro.xacro (robot description, xacro)
@@ -15,10 +15,11 @@
 				</geometry>
 			</visual>
-			<collision>
+                        <!-- This collision link is broken and not proper, it prevents the whole gripper from being used in MoveIt! -->
+			<!-- <collision>
 				<origin xyz="-0.0455 0.0414 0.036" rpy="0 3.1416 -1.57"/>
 				<geometry>
 					<mesh filename="package://robotiq_s_model_visualization/meshes/s-model_articulated/collision/link_0.STL" />
 				</geometry>
-			</collision>
+			</collision> -->
             <inertial>
                 <origin xyz="0 0 0" rpy="0 0 0"/>

Commit message: sigh

File: robotiq_s_model_visualization/cfg/s-model_articulated_macro.xacro (robot description, xacro)
@@ -21,5 +21,5 @@
 				</geometry>
 			</visual>
-			<collision>
+			 <collision>
 				<geometry>
 					<mesh filename="package://robotiq_s_model_visualization/meshes/s-model_articulated/collision/palm.STL" />
@@ -29,4 +29,5 @@
                 <gazebo reference="${prefix}palm">
                         <material>Gazebo/Blue</material>
+                        <selfCollide>true</selfCollide>
                 </gazebo>
         <inertial>

File: robotiq_s_model_visualization/cfg/s-model_finger_articulated_macro.xacro (robot description, xacro)
@@ -16,10 +16,10 @@
 			</visual>
                         <!-- This collision link is broken and not proper, it prevents the whole gripper from being used in MoveIt! -->
-			<!-- <collision>
+			<collision>
 				<origin xyz="-0.0455 0.0414 0.036" rpy="0 3.1416 -1.57"/>
 				<geometry>
 					<mesh filename="package://robotiq_s_model_visualization/meshes/s-model_articulated/collision/link_0.STL" />
 				</geometry>
-			</collision> -->
+			</collision>
             <inertial>
                 <origin xyz="0 0 0" rpy="0 0 0"/>
@@ -30,5 +30,5 @@
                 <gazebo reference="${prefix}link_0">
                     <material>Gazebo/Black</material>
-                    <selfCollide>false</selfCollide>
+                    <selfCollide>true</selfCollide>
                 </gazebo>
 		<link name="${prefix}link_1">
@@ -39,5 +39,5 @@
 				</geometry>
 			</visual>
-			<collision>
+			 <collision>
 				<origin xyz="0.050 -.028 0" rpy="0 0 -0.52"/>
 				<geometry>
@@ -53,5 +53,5 @@
                  <gazebo reference="${prefix}link_1">
                             <material>Gazebo/Black</material>
-                            <selfCollide>false</selfCollide>
+                            <selfCollide>true</selfCollide>
                  </gazebo>
 		<link name="${prefix}link_2">
@@ -67,5 +67,5 @@
 				</geometry>
 			</visual>
-			<collision>
+			 <collision>
 				<origin xyz="0.039 0 0.0075" rpy="0 0 0"/>
 				<geometry>
@@ -81,5 +81,5 @@
  <gazebo reference="${prefix}link_2">
 				<material>Gazebo/Black</material>
-                                <selfCollide>false</selfCollide>
+                                <selfCollide>true</selfCollide>
                                 </gazebo>
 		<link name="${prefix}link_3">
@@ -90,5 +90,5 @@
 				</geometry>
 			</visual>
-			<collision>
+			 <collision>
 				<origin xyz="0 0 0" rpy="0 0 0.52"/>
 				<geometry>
@@ -104,5 +104,5 @@
 <gazebo reference="${prefix}link_2">
 				<material>Gazebo/Black</material>
-                                <selfCollide>false</selfCollide>
+                                <selfCollide>true</selfCollide>
                                 </gazebo>
 		<!-- end of link list -->

Commit message: Added working xacro

File: robotiq_s_model_visualization/cfg/s-model_articulated_macro.xacro (robot description, xacro)
@@ -5,9 +5,5 @@
 there are multiple hands then a prefix followed by an "_" is needed.
 -->
-        <!-- Gazebo plugin for ROS Control -->
-        <!-- <gazebo>
-            <plugin name="ros_control" filename="libgazebo_ros_control.so"/>
--->
-<robot xmlns:xacro="http://ros.org/wiki/xacro">
+<robot xmlns:xacro="http://ros.org/wiki/xacro" name="tests">
 	<xacro:include filename="$(find robotiq_s_model_visualization)/cfg/s-model_finger_articulated_macro.xacro" />
 	<xacro:macro name="s-model_articulated" params="prefix">
@@ -15,4 +11,5 @@
 	<xacro:s-model_finger_articulated prefix="${prefix}finger_2_"/>
 	<xacro:s-model_finger_articulated prefix="${prefix}finger_middle_"/>
+		<!-- link list -->
 		<link name="${prefix}palm">
 			<visual>
@@ -20,15 +17,17 @@
 					<mesh filename="package://robotiq_s_model_visualization/meshes/s-model_articulated/visual/palm.STL" />
 				</geometry>
+				<material name="green">
+					<color rgba="0 1 0 1"/>
+				</material>
 			</visual>
-			 <collision>
+			<collision>
 				<geometry>
 					<mesh filename="package://robotiq_s_model_visualization/meshes/s-model_articulated/collision/palm.STL" />
 				</geometry>
+				<material name="yellow">
+					<color rgba="0 1 1 1"/>
+				</material>
 			</collision>
 		</link>
-                <gazebo reference="${prefix}palm">
-                        <material>Gazebo/Blue</material>
-                        <selfCollide>true</selfCollide>
-                </gazebo>
         <inertial>
             <origin xyz="0 0 0" rpy="0 0 0"/>
@@ -45,5 +44,6 @@
 			<origin xyz="-0.0455 0.0214 0.036" rpy="0 3.1416 -1.57"/>
 			<limit lower="-0.16" upper="0.25" effort="100" velocity="100"/>
-                </joint>
+		</joint>
+		<!-- WARNING: LIMITS NOT CORRECT -->
 		<joint name="${prefix}palm_finger_2_joint" type="revolute">
 			<parent link="${prefix}palm"/>
@@ -59,4 +59,6 @@
 			<origin xyz="0.0455 0.0214 0" rpy="0 0 1.57"/>
 		</joint>
+		<!-- end of joint list -->
 	</xacro:macro>
+     <xacro:s-model_articulated prefix=""/>
 </robot>

File: robotiq_s_model_visualization/cfg/s-model_finger_articulated_macro.xacro (robot description, xacro)
@@ -14,6 +14,8 @@
 					<mesh filename="package://robotiq_s_model_visualization/meshes/s-model_articulated/visual/link_0.STL" />
 				</geometry>
+				<material name="green">
+					<color rgba="0 1 0 1"/>
+				</material>
 			</visual>
-                        <!-- This collision link is broken and not proper, it prevents the whole gripper from being used in MoveIt! -->
 			<collision>
 				<origin xyz="-0.0455 0.0414 0.036" rpy="0 3.1416 -1.57"/>
@@ -21,4 +23,7 @@
 					<mesh filename="package://robotiq_s_model_visualization/meshes/s-model_articulated/collision/link_0.STL" />
 				</geometry>
+				<material name="yellow">
+					<color rgba="0 1 1 1"/>
+				</material>
 			</collision>
             <inertial>
@@ -28,8 +33,4 @@
             </inertial>
 		</link>
-                <gazebo reference="${prefix}link_0">
-                    <material>Gazebo/Black</material>
-                    <selfCollide>true</selfCollide>
-                </gazebo>
 		<link name="${prefix}link_1">
 			<visual>
@@ -38,10 +39,12 @@
 					<mesh filename="package://robotiq_s_model_visualization/meshes/s-model_articulated/visual/link_1.STL" />
 				</geometry>
+				<material name="green"/>
 			</visual>
-			 <collision>
+			<collision>
 				<origin xyz="0.050 -.028 0" rpy="0 0 -0.52"/>
 				<geometry>
 					<mesh filename="package://robotiq_s_model_visualization/meshes/s-model_articulated/collision/link_1.STL" />
 				</geometry>
+				<material name="yellow"/>
 			</collision>
             <inertial>
@@ -51,8 +54,4 @@
             </inertial>
 		</link>
-                 <gazebo reference="${prefix}link_1">
-                            <material>Gazebo/Black</material>
-                            <selfCollide>true</selfCollide>
-                 </gazebo>
 		<link name="${prefix}link_2">
 			<!--
@@ -66,10 +65,12 @@
 					<mesh filename="package://robotiq_s_model_visualization/meshes/s-model_articulated/visual/link_2.STL" />
 				</geometry>
+				<material name="green"/>
 			</visual>
-			 <collision>
+			<collision>
 				<origin xyz="0.039 0 0.0075" rpy="0 0 0"/>
 				<geometry>
 					<mesh filename="package://robotiq_s_model_visualization/meshes/s-model_articulated/collision/link_2.STL" />
 				</geometry>
+				<material name="yellow"/>
 			</collision>
             <inertial>
@@ -79,8 +80,4 @@
             </inertial>
 		</link>
- <gazebo reference="${prefix}link_2">
-				<material>Gazebo/Black</material>
-                                <selfCollide>true</selfCollide>
-                                </gazebo>
 		<link name="${prefix}link_3">
 			<visual>
@@ -89,10 +86,12 @@
 					<mesh filename="package://robotiq_s_model_visualization/meshes/s-model_articulated/visual/link_3.STL" />
 				</geometry>
+				<material name="green"/>
 			</visual>
-			 <collision>
+			<collision>
 				<origin xyz="0 0 0" rpy="0 0 0.52"/>
 				<geometry>
 					<mesh filename="package://robotiq_s_model_visualization/meshes/s-model_articulated/collision/link_3.STL" />
 				</geometry>
+				<material name="yellow"/>
 			</collision>
             <inertial>
@@ -102,8 +101,4 @@
             </inertial>
 		</link>
-<gazebo reference="${prefix}link_2">
-				<material>Gazebo/Black</material>
-                                <selfCollide>true</selfCollide>
-                                </gazebo>
 		<!-- end of link list -->
 		<!-- joint list -->

File: robotiq_s_model_visualization/cfg/s-model_mesh_macro.xacro (robot description, xacro)
@@ -1,3 +1,3 @@
-<robot xmlns:xacro="http://ros.org/wiki/xacro">
+<robot xmlns:xacro="http://ros.org/wiki/xacro" name="joops">
 	<xacro:macro name="s-model_mesh" params="prefix">
 		<!-- link list -->
@@ -81,3 +81,4 @@
 		<!-- end of joint list -->
 	</xacro:macro>
+       <xacro:s-model_mesh prefix=""/>
 </robot>
