Commit message: Cleanup of the robotiq package. Includes removing boiler plates, capitalization, removing whitespace, removing unneeded files, etc.
Add the robotiq_s_model_articulated_gazebo package.

Added self collide for finger links

Added

Fixed inertial tag

fixed things

Added gazebo plugin for s-model_articulated

Added messages and gazebo plugin

Updated namespaces w.r.t changes of externalizing package

Added things to CMake so it compiles

Added gazebo pkg

Added the gazebo pkg

ok

Why u no build..

damnit gazebo

Apparently gazebo parses things that are commented out. Go figure

Removed unneeded args in launch file

Renamed robot to-> gripper

Modified package.xml in gazebo_plugins to be apache 2.0

Added modifier declaration to .h

Fixed whitespace

Removed boilerplates from CMakeLists

Removed more boilerplate CMakeLists text

Removed unnecessary variable directing of {PROJECT_SOURCE_DIR}

Removed old directory with wrong name under /include

Removed unnecessary message installation via INSTALL

Removed unnecessary files from PR

Renamed joops to s-model_mesh

Removed macro in file that was only there for testing

Capitlization of Robotiq

No longer requires dependency on _EXPORTED_TARGETS

Capitlization of Robotiq

Added comment explaining private member accessing

Removed instantiation of robotiq_hand.urdf.xacro, poor design

Made xacro instantiation file for robotiq_s_model

File: robotiq_s_model_visualization/cfg/s-model_articulated_macro.xacro (robot description, xacro)
@@ -29,10 +29,10 @@
 				</material>
 			</collision>
+		<inertial>
+		    <origin xyz="0 0 0" rpy="0 0 0"/>
+		    <mass value="1.3"/>
+		    <inertia ixx="0.006012" ixy="0.000079" ixz="-0.00024" iyy="0.012892" iyz="0" izz="0.002435" />
+		</inertial>
 		</link>
-        <inertial>
-            <origin xyz="0 0 0" rpy="0 0 0"/>
-            <mass value="1.3"/>
-            <inertia ixx="0.006012" ixy="0.000079" ixz="-0.00024" iyy="0.012892" iyz="0" izz="0.002435" />
-        </inertial>
 		<!-- end of link list -->
 		<!-- joint list -->
@@ -53,9 +53,12 @@
 			<limit lower="-0.25" upper="0.16" effort="100" velocity="100"/>
 		</joint>
-		<joint name="${prefix}palm_finger_middle_joint" type="fixed">
+                <!-- WARNING: LIMITS NOT CORRECT -->
+                <!-- Changed to revolute so gazebo doesn't flip tables -->
+		<joint name="${prefix}palm_finger_middle_joint" type="revolute">
 			<parent link="${prefix}palm"/>
 			<child link="${prefix}finger_middle_link_0"/>
 			<axis xyz="0 0 1"/>
 			<origin xyz="0.0455 0.0214 0" rpy="0 0 1.57"/>
+                        <limit lower="-0.25" upper="0.16" effort="100" velocity="100"/>
 		</joint>
 		<!-- end of joint list -->

File: robotiq_s_model_visualization/cfg/s-model_mesh_macro.xacro (robot description, xacro)
@@ -1,3 +1,3 @@
-<robot xmlns:xacro="http://ros.org/wiki/xacro" name="joops">
+<robot xmlns:xacro="http://ros.org/wiki/xacro" name="s-model_mesh">
 	<xacro:macro name="s-model_mesh" params="prefix">
 		<!-- link list -->
@@ -81,4 +81,3 @@
 		<!-- end of joint list -->
 	</xacro:macro>
-       <xacro:s-model_mesh prefix=""/>
 </robot>

Commit message: Fixed inertial tag

File: robotiq_s_model_visualization/cfg/s-model_articulated_macro.xacro (robot description, xacro)
@@ -29,10 +29,10 @@
 				</material>
 			</collision>
+		<inertial>
+		    <origin xyz="0 0 0" rpy="0 0 0"/>
+		    <mass value="1.3"/>
+		    <inertia ixx="0.006012" ixy="0.000079" ixz="-0.00024" iyy="0.012892" iyz="0" izz="0.002435" />
+		</inertial>
 		</link>
-        <inertial>
-            <origin xyz="0 0 0" rpy="0 0 0"/>
-            <mass value="1.3"/>
-            <inertia ixx="0.006012" ixy="0.000079" ixz="-0.00024" iyy="0.012892" iyz="0" izz="0.002435" />
-        </inertial>
 		<!-- end of link list -->
 		<!-- joint list -->

Commit message: fixed things

File: robotiq_s_model_visualization/cfg/s-model_articulated_macro.xacro (robot description, xacro)
@@ -53,9 +53,12 @@
 			<limit lower="-0.25" upper="0.16" effort="100" velocity="100"/>
 		</joint>
-		<joint name="${prefix}palm_finger_middle_joint" type="fixed">
+                <!-- WARNING: LIMITS NOT CORRECT -->
+                <!-- Changed to revolute so gazebo doesn't flip tables -->
+		<joint name="${prefix}palm_finger_middle_joint" type="revolute">
 			<parent link="${prefix}palm"/>
 			<child link="${prefix}finger_middle_link_0"/>
 			<axis xyz="0 0 1"/>
 			<origin xyz="0.0455 0.0214 0" rpy="0 0 1.57"/>
+                        <limit lower="-0.25" upper="0.16" effort="100" velocity="100"/>
 		</joint>
 		<!-- end of joint list -->

Commit message: added dual ur5 stuff

File: robotiq_s_model_visualization/cfg/s-model_articulated_macro.xacro (robot description, xacro)
@@ -17,6 +17,6 @@
 					<mesh filename="package://robotiq_s_model_visualization/meshes/s-model_articulated/visual/palm.STL" />
 				</geometry>
-				<material name="gray">
-					<color rgba="0.2 0.2 0.2 1"/>
+				<material name="green">
+					<color rgba="0 1 0 1"/>
 				</material>
 			</visual>

File: robotiq_s_model_visualization/cfg/s-model_finger_articulated_macro.xacro (robot description, xacro)
@@ -14,6 +14,6 @@
 					<mesh filename="package://robotiq_s_model_visualization/meshes/s-model_articulated/visual/link_0.STL" />
 				</geometry>
-				<material name="gray">
-					<color rgba="0.2 0.2 0.2 1"/>
+				<material name="green">
+					<color rgba="0 1 0 1"/>
 				</material>
 			</visual>
@@ -39,5 +39,5 @@
 					<mesh filename="package://robotiq_s_model_visualization/meshes/s-model_articulated/visual/link_1.STL" />
 				</geometry>
-				<material name="gray"/>
+				<material name="green"/>
 			</visual>
 			<collision>
@@ -65,5 +65,5 @@
 					<mesh filename="package://robotiq_s_model_visualization/meshes/s-model_articulated/visual/link_2.STL" />
 				</geometry>
-				<material name="gray"/>
+				<material name="green"/>
 			</visual>
 			<collision>
@@ -86,5 +86,5 @@
 					<mesh filename="package://robotiq_s_model_visualization/meshes/s-model_articulated/visual/link_3.STL" />
 				</geometry>
-				<material name="gray"/>
+				<material name="green"/>
 			</visual>
 			<collision>

Commit message: fix the bug where gazebo launch does not work due to missing upload.launch in urdf

File: robotiq_s_model_visualization/cfg/s-model_articulated_macro.xacro (robot description, xacro)
@@ -17,6 +17,6 @@
 					<mesh filename="package://robotiq_s_model_visualization/meshes/s-model_articulated/visual/palm.STL" />
 				</geometry>
-				<material name="gray">
-					<color rgba="0.2 0.2 0.2 1"/>
+				<material name="green">
+					<color rgba="0 1 0 1"/>
 				</material>
 			</visual>
@@ -29,13 +29,13 @@
 				</material>
 			</collision>
+		<inertial>
+		    <origin xyz="0 0 0" rpy="0 0 0"/>
+		    <mass value="1.3"/>
+		    <inertia ixx="0.006012" ixy="0.000079" ixz="-0.00024" iyy="0.012892" iyz="0" izz="0.002435" />
+		</inertial>
 		</link>
-		<link name="${prefix}tool0"/>
-        <inertial>
-            <origin xyz="0 0 0" rpy="0 0 0"/>
-            <mass value="1.3"/>
-            <inertia ixx="0.006012" ixy="0.000079" ixz="-0.00024" iyy="0.012892" iyz="0" izz="0.002435" />
-        </inertial>
 		<!-- end of link list -->
 		<!-- joint list -->
+		<!-- WARNING: LIMITS NOT CORRECT -->
 		<joint name="${prefix}palm_finger_1_joint" type="revolute">
 			<parent link="${prefix}palm"/>
@@ -43,6 +43,7 @@
 			<axis xyz="0 1 0"/>
 			<origin xyz="-0.0455 0.0214 0.036" rpy="0 3.1416 -1.57"/>
-			<limit lower="-0.1784" upper="0.192" effort="100" velocity="100"/>
+			<limit lower="-0.16" upper="0.25" effort="100" velocity="100"/>
 		</joint>
+		<!-- WARNING: LIMITS NOT CORRECT -->
 		<joint name="${prefix}palm_finger_2_joint" type="revolute">
 			<parent link="${prefix}palm"/>
@@ -50,16 +51,14 @@
 			<axis xyz="0 1 0"/>
 			<origin xyz="-0.0455 0.0214 -0.036" rpy="0 3.1416 -1.57"/>
-			<limit lower="-0.192" upper="0.1784" effort="100" velocity="100"/>
+			<limit lower="-0.25" upper="0.16" effort="100" velocity="100"/>
 		</joint>
-		<joint name="${prefix}palm_finger_middle_joint" type="fixed">
+                <!-- WARNING: LIMITS NOT CORRECT -->
+                <!-- Changed to revolute so gazebo doesn't flip tables -->
+		<joint name="${prefix}palm_finger_middle_joint" type="revolute">
 			<parent link="${prefix}palm"/>
 			<child link="${prefix}finger_middle_link_0"/>
 			<axis xyz="0 0 1"/>
 			<origin xyz="0.0455 0.0214 0" rpy="0 0 1.57"/>
-		</joint>
-		<joint name="${prefix}palm_tool0" type="fixed">
-			<parent link="${prefix}palm"/>
-			<child link="${prefix}tool0"/>
-			<origin xyz="0.0 0.0875 0.0" rpy="0 0 1.5707"/>
+                        <limit lower="-0.25" upper="0.16" effort="100" velocity="100"/>
 		</joint>
 		<!-- end of joint list -->

File: robotiq_s_model_visualization/cfg/s-model_finger_articulated_macro.xacro (robot description, xacro)
@@ -14,10 +14,10 @@
 					<mesh filename="package://robotiq_s_model_visualization/meshes/s-model_articulated/visual/link_0.STL" />
 				</geometry>
-				<material name="gray">
-					<color rgba="0.2 0.2 0.2 1"/>
+				<material name="green">
+					<color rgba="0 1 0 1"/>
 				</material>
 			</visual>
 			<collision>
-				<origin xyz="0.020 0 0" rpy="0 0 0"/>
+				<origin xyz="-0.0455 0.0414 0.036" rpy="0 3.1416 -1.57"/>
 				<geometry>
 					<mesh filename="package://robotiq_s_model_visualization/meshes/s-model_articulated/collision/link_0.STL" />
@@ -39,5 +39,5 @@
 					<mesh filename="package://robotiq_s_model_visualization/meshes/s-model_articulated/visual/link_1.STL" />
 				</geometry>
-				<material name="gray"/>
+				<material name="green"/>
 			</visual>
 			<collision>
@@ -65,5 +65,5 @@
 					<mesh filename="package://robotiq_s_model_visualization/meshes/s-model_articulated/visual/link_2.STL" />
 				</geometry>
-				<material name="gray"/>
+				<material name="green"/>
 			</visual>
 			<collision>
@@ -86,5 +86,5 @@
 					<mesh filename="package://robotiq_s_model_visualization/meshes/s-model_articulated/visual/link_3.STL" />
 				</geometry>
-				<material name="gray"/>
+				<material name="green"/>
 			</visual>
 			<collision>
@@ -103,4 +103,5 @@
 		<!-- end of link list -->
 		<!-- joint list -->
+		<!-- WARNING: LIMITS NOT CORRECT -->
 		<joint name="${prefix}joint_1" type="revolute">
 			<parent link="${prefix}link_0"/>
@@ -108,6 +109,7 @@
 			<axis xyz="0 0 1"/>
 			<origin xyz="0.020 0 0" rpy="0 0 0"/>
-			<limit lower="0.0495" upper="1.2218" effort="100" velocity="100"/>
+			<limit lower="0" upper="3.1416" effort="100" velocity="100"/>
 		</joint>
+		<!-- WARNING: LIMITS NOT CORRECT -->
 		<joint name="${prefix}joint_2" type="revolute">
 			<parent link="${prefix}link_1"/>
@@ -115,6 +117,7 @@
 			<axis xyz="0 0 1"/>
 			<origin xyz="0.050 -.028 0" rpy="0 0 -0.52"/>
-			<limit lower="0.0" upper="1.5708" effort="100" velocity="100"/>
+			<limit lower="0" upper="3.1416" effort="100" velocity="100"/>
 		</joint>
+		<!-- WARNING: LIMITS NOT CORRECT -->
 		<joint name="${prefix}joint_3" type="revolute">
 			<parent link="${prefix}link_2"/>
@@ -122,5 +125,5 @@
 			<axis xyz="0 0 1"/>
 			<origin xyz="0.039 0 0" rpy="0 0 0"/>
-			<limit lower="-1.2217" upper="-0.0523" effort="100" velocity="100"/>
+			<limit lower="0" upper="3.1416" effort="100" velocity="100"/>
 		</joint>
 		<!-- end of joint list -->

Commit message: merge the new mesh and urdf from indigo-dev branch of robotiq

File: robotiq_s_model_visualization/cfg/s-model_articulated_macro.xacro (robot description, xacro)
@@ -17,6 +17,6 @@
 					<mesh filename="package://robotiq_s_model_visualization/meshes/s-model_articulated/visual/palm.STL" />
 				</geometry>
-				<material name="green">
-					<color rgba="0 1 0 1"/>
+				<material name="gray">
+					<color rgba="0.2 0.2 0.2 1"/>
 				</material>
 			</visual>
@@ -29,13 +29,13 @@
 				</material>
 			</collision>
-		<inertial>
-		    <origin xyz="0 0 0" rpy="0 0 0"/>
-		    <mass value="1.3"/>
-		    <inertia ixx="0.006012" ixy="0.000079" ixz="-0.00024" iyy="0.012892" iyz="0" izz="0.002435" />
-		</inertial>
 		</link>
+		<link name="${prefix}tool0"/>
+        <inertial>
+            <origin xyz="0 0 0" rpy="0 0 0"/>
+            <mass value="1.3"/>
+            <inertia ixx="0.006012" ixy="0.000079" ixz="-0.00024" iyy="0.012892" iyz="0" izz="0.002435" />
+        </inertial>
 		<!-- end of link list -->
 		<!-- joint list -->
-		<!-- WARNING: LIMITS NOT CORRECT -->
 		<joint name="${prefix}palm_finger_1_joint" type="revolute">
 			<parent link="${prefix}palm"/>
@@ -43,7 +43,6 @@
 			<axis xyz="0 1 0"/>
 			<origin xyz="-0.0455 0.0214 0.036" rpy="0 3.1416 -1.57"/>
-			<limit lower="-0.16" upper="0.25" effort="100" velocity="100"/>
+			<limit lower="-0.1784" upper="0.192" effort="100" velocity="100"/>
 		</joint>
-		<!-- WARNING: LIMITS NOT CORRECT -->
 		<joint name="${prefix}palm_finger_2_joint" type="revolute">
 			<parent link="${prefix}palm"/>
@@ -51,14 +50,16 @@
 			<axis xyz="0 1 0"/>
 			<origin xyz="-0.0455 0.0214 -0.036" rpy="0 3.1416 -1.57"/>
-			<limit lower="-0.25" upper="0.16" effort="100" velocity="100"/>
+			<limit lower="-0.192" upper="0.1784" effort="100" velocity="100"/>
 		</joint>
-                <!-- WARNING: LIMITS NOT CORRECT -->
-                <!-- Changed to revolute so gazebo doesn't flip tables -->
-		<joint name="${prefix}palm_finger_middle_joint" type="revolute">
+		<joint name="${prefix}palm_finger_middle_joint" type="fixed">
 			<parent link="${prefix}palm"/>
 			<child link="${prefix}finger_middle_link_0"/>
 			<axis xyz="0 0 1"/>
 			<origin xyz="0.0455 0.0214 0" rpy="0 0 1.57"/>
-                        <limit lower="-0.25" upper="0.16" effort="100" velocity="100"/>
+		</joint>
+		<joint name="${prefix}palm_tool0" type="fixed">
+			<parent link="${prefix}palm"/>
+			<child link="${prefix}tool0"/>
+			<origin xyz="0.0 0.0875 0.0" rpy="0 0 1.5707"/>
 		</joint>
 		<!-- end of joint list -->

File: robotiq_s_model_visualization/cfg/s-model_finger_articulated_macro.xacro (robot description, xacro)
@@ -14,10 +14,10 @@
 					<mesh filename="package://robotiq_s_model_visualization/meshes/s-model_articulated/visual/link_0.STL" />
 				</geometry>
-				<material name="green">
-					<color rgba="0 1 0 1"/>
+				<material name="gray">
+					<color rgba="0.2 0.2 0.2 1"/>
 				</material>
 			</visual>
 			<collision>
-				<origin xyz="-0.0455 0.0414 0.036" rpy="0 3.1416 -1.57"/>
+				<origin xyz="0.020 0 0" rpy="0 0 0"/>
 				<geometry>
 					<mesh filename="package://robotiq_s_model_visualization/meshes/s-model_articulated/collision/link_0.STL" />
@@ -39,5 +39,5 @@
 					<mesh filename="package://robotiq_s_model_visualization/meshes/s-model_articulated/visual/link_1.STL" />
 				</geometry>
-				<material name="green"/>
+				<material name="gray"/>
 			</visual>
 			<collision>
@@ -65,5 +65,5 @@
 					<mesh filename="package://robotiq_s_model_visualization/meshes/s-model_articulated/visual/link_2.STL" />
 				</geometry>
-				<material name="green"/>
+				<material name="gray"/>
 			</visual>
 			<collision>
@@ -86,5 +86,5 @@
 					<mesh filename="package://robotiq_s_model_visualization/meshes/s-model_articulated/visual/link_3.STL" />
 				</geometry>
-				<material name="green"/>
+				<material name="gray"/>
 			</visual>
 			<collision>
@@ -103,5 +103,4 @@
 		<!-- end of link list -->
 		<!-- joint list -->
-		<!-- WARNING: LIMITS NOT CORRECT -->
 		<joint name="${prefix}joint_1" type="revolute">
 			<parent link="${prefix}link_0"/>
@@ -109,7 +108,6 @@
 			<axis xyz="0 0 1"/>
 			<origin xyz="0.020 0 0" rpy="0 0 0"/>
-			<limit lower="0" upper="3.1416" effort="100" velocity="100"/>
+			<limit lower="0.0495" upper="1.2218" effort="100" velocity="100"/>
 		</joint>
-		<!-- WARNING: LIMITS NOT CORRECT -->
 		<joint name="${prefix}joint_2" type="revolute">
 			<parent link="${prefix}link_1"/>
@@ -117,7 +115,6 @@
 			<axis xyz="0 0 1"/>
 			<origin xyz="0.050 -.028 0" rpy="0 0 -0.52"/>
-			<limit lower="0" upper="3.1416" effort="100" velocity="100"/>
+			<limit lower="0.0" upper="1.5708" effort="100" velocity="100"/>
 		</joint>
-		<!-- WARNING: LIMITS NOT CORRECT -->
 		<joint name="${prefix}joint_3" type="revolute">
 			<parent link="${prefix}link_2"/>
@@ -125,5 +122,5 @@
 			<axis xyz="0 0 1"/>
 			<origin xyz="0.039 0 0" rpy="0 0 0"/>
-			<limit lower="0" upper="3.1416" effort="100" velocity="100"/>
+			<limit lower="-1.2217" upper="-0.0523" effort="100" velocity="100"/>
 		</joint>
 		<!-- end of joint list -->

File: robotiq_s_model_visualization/cfg/s-model_mesh_macro.xacro (robot description, xacro)
@@ -1,3 +1,3 @@
-<robot xmlns:xacro="http://ros.org/wiki/xacro" name="s-model_mesh">
+<robot xmlns:xacro="http://ros.org/wiki/xacro">
 	<xacro:macro name="s-model_mesh" params="prefix">
 		<!-- link list -->
