Commit message: Reduced mesh file path length to fix assimp error

File: robotiq_c2_model_visualization/urdf/robotiq_c2_model.urdf (robot description, URDF)
Before this commit: robot robotiq_c2_model, 10 links, 9 joints
Links:
- link robotiq_85_adapter_link: geometry collision mesh filename=package://robotiq_c2_model_visualization/meshes/collision/r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; visual mesh filename=package://robotiq_c2_model_visualization/meshes/visual/robo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
- link robotiq_85_base_link: geometry collision mesh filename=package://robotiq_c2_model_visualization/meshes/collision/r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; visual mesh filename=package://robotiq_c2_model_visualization/meshes/visual/robo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
- link robotiq_85_left_finger_link: geometry collision mesh filename=package://robotiq_c2_model_visualization/meshes/collision/r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; visual mesh filename=package://robotiq_c2_model_visualization/meshes/visual/robo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
- link robotiq_85_left_finger_tip_link: geometry collision mesh filename=package://robotiq_c2_model_visualization/meshes/collision/r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; visual mesh filename=package://robotiq_c2_model_visualization/meshes/visual/robo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
- link robotiq_85_left_inner_knuckle_link: geometry collision mesh filename=package://robotiq_c2_model_visualization/meshes/collision/r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; visual mesh filename=package://robotiq_c2_model_visualization/meshes/visual/robo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
- link robotiq_85_left_knuckle_link: geometry collision mesh filename=package://robotiq_c2_model_visualization/meshes/collision/r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; visual mesh filename=package://robotiq_c2_model_visualization/meshes/visual/robo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
- link robotiq_85_right_finger_link: geometry collision mesh filename=package://robotiq_c2_model_visualization/meshes/collision/r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; visual mesh filename=package://robotiq_c2_model_visualization/meshes/visual/robo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
- link robotiq_85_right_finger_tip_link: geometry collision mesh filename=package://robotiq_c2_model_visualization/meshes/collision/r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; visual mesh filename=package://robotiq_c2_model_visualization/meshes/visual/robo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
- link robotiq_85_right_inner_knuckle_link: geometry collision mesh filename=package://robotiq_c2_model_visualization/meshes/collision/r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; visual mesh filename=package://robotiq_c2_model_visualization/meshes/visual/robo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
- link robotiq_85_right_knuckle_link: geometry collision mesh filename=package://robotiq_c2_model_visualization/meshes/collision/r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; visual mesh filename=package://robotiq_c2_model_visualization/meshes/visual/robo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

File: robotiq_c2_model_visualization/urdf/robotiq_c2_model_macro.xacro (robot description, xacro)
@@ -11,5 +11,5 @@
     <visual>
       <geometry>
-        <mesh filename="package://robotiq_c2_model_visualization/meshes/robotiq_c2/visual/robotiq_85_gripper_adapter_plate.dae"/>
+        <mesh filename="package://robotiq_c2_model_visualization/meshes/visual/robotiq_85_gripper_adapter_plate.dae"/>
       </geometry>
       <origin rpy="1.5707 0 1.5707" xyz="0 0 0"/>
@@ -17,5 +17,5 @@
     <collision>
       <geometry>
-        <mesh filename="package://robotiq_c2_model_visualization/meshes/robotiq_c2/collision/robotiq_85_gripper_adapter_plate.dae"/>
+        <mesh filename="package://robotiq_c2_model_visualization/meshes/collision/robotiq_85_gripper_adapter_plate.dae"/>
       </geometry>
       <origin rpy="0 0 1.5707" xyz="0 0 0"/>
@@ -33,5 +33,5 @@
     <visual>
       <geometry>
-        <mesh filename="package://robotiq_c2_model_visualization/meshes/robotiq_c2/visual/robotiq_85_gripper_base.dae"/>
+        <mesh filename="package://robotiq_c2_model_visualization/meshes/visual/robotiq_85_gripper_base.dae"/>
       </geometry>
       <origin rpy="3.1415 0 1.5707" xyz="0 0 0"/>
@@ -39,5 +39,5 @@
     <collision>
       <geometry>
-        <mesh filename="package://robotiq_c2_model_visualization/meshes/robotiq_c2/collision/robotiq_85_gripper_base.dae"/>
+        <mesh filename="package://robotiq_c2_model_visualization/meshes/collision/robotiq_85_gripper_base.dae"/>
       </geometry>
       <origin rpy="1.5707 0 1.5707" xyz="0 0 0"/>
@@ -66,5 +66,5 @@
     <visual>
       <geometry>
-        <mesh filename="package://robotiq_c2_model_visualization/meshes/robotiq_c2/visual/robotiq_85_gripper_joint_0_L.dae"/>
+        <mesh filename="package://robotiq_c2_model_visualization/meshes/visual/robotiq_85_gripper_joint_0_L.dae"/>
       </geometry>
       <origin rpy="3.14159 -1.5707 0" xyz="0 .04191 -.0306"/>
@@ -72,5 +72,5 @@
     <collision>
       <geometry>
-        <mesh filename="package://robotiq_c2_model_visualization/meshes/robotiq_c2/collision/robotiq_85_gripper_joint_0_L.dae"/>
+        <mesh filename="package://robotiq_c2_model_visualization/meshes/collision/robotiq_85_gripper_joint_0_L.dae"/>
       </geometry>
       <origin rpy="1.5707 -1.5707 0" xyz="0 .04191 -.0306"/>
@@ -80,5 +80,5 @@
     <visual>
       <geometry>
-        <mesh filename="package://robotiq_c2_model_visualization/meshes/robotiq_c2/visual/robotiq_85_gripper_joint_0_R.dae"/>
+        <mesh filename="package://robotiq_c2_model_visualization/meshes/visual/robotiq_85_gripper_joint_0_R.dae"/>
       </geometry>
       <origin rpy="3.14159 1.5707 0" xyz="0 .04191 -.0306"/>
@@ -86,5 +86,5 @@
     <collision>
       <geometry>
-        <mesh filename="package://robotiq_c2_model_visualization/meshes/robotiq_c2/collision/robotiq_85_gripper_joint_0_R.dae"/>
+        <mesh filename="package://robotiq_c2_model_visualization/meshes/collision/robotiq_85_gripper_joint_0_R.dae"/>
       </geometry>
       <origin rpy="1.5707 1.5707 0" xyz="0 .04191 -.0306"/>
@@ -112,5 +112,5 @@
     <visual>
       <geometry>
-        <mesh filename="package://robotiq_c2_model_visualization/meshes/robotiq_c2/visual/robotiq_85_gripper_joint_1_L.dae"/>
+        <mesh filename="package://robotiq_c2_model_visualization/meshes/visual/robotiq_85_gripper_joint_1_L.dae"/>
       </geometry>
       <origin rpy="0 1.5707 0" xyz="0 -.03683 .06194"/>
@@ -118,5 +118,5 @@
     <collision>
       <geometry>
-        <mesh filename="package://robotiq_c2_model_visualization/meshes/robotiq_c2/collision/robotiq_85_gripper_joint_1_L.dae"/>
+        <mesh filename="package://robotiq_c2_model_visualization/meshes/collision/robotiq_85_gripper_joint_1_L.dae"/>
       </geometry>
       <origin rpy="-1.5707 1.5707 0" xyz="0 -.03683 .06194"/>
@@ -126,5 +126,5 @@
     <visual>
       <geometry>
-        <mesh filename="package://robotiq_c2_model_visualization/meshes/robotiq_c2/visual/robotiq_85_gripper_joint_1_R.dae"/>
+        <mesh filename="package://robotiq_c2_model_visualization/meshes/visual/robotiq_85_gripper_joint_1_R.dae"/>
       </geometry>
       <origin rpy="0 -1.5707 0" xyz="0 -.03683 .06194"/>
@@ -132,5 +132,5 @@
     <collision>
       <geometry>
-        <mesh filename="package://robotiq_c2_model_visualization/meshes/robotiq_c2/collision/robotiq_85_gripper_joint_1_R.dae"/>
+        <mesh filename="package://robotiq_c2_model_visualization/meshes/collision/robotiq_85_gripper_joint_1_R.dae"/>
       </geometry>
       <origin rpy="-1.5707 -1.5707 0" xyz="0 -.03683 .06194"/>
@@ -160,5 +160,5 @@
     <visual>
       <geometry>
-        <mesh filename="package://robotiq_c2_model_visualization/meshes/robotiq_c2/visual/robotiq_85_gripper_joint_2_L.dae"/>
+        <mesh filename="package://robotiq_c2_model_visualization/meshes/visual/robotiq_85_gripper_joint_2_L.dae"/>
       </geometry>
       <origin rpy="0 1.5707 0" xyz="0 -.04843 .0127"/>
@@ -166,5 +166,5 @@
     <collision>
       <geometry>
-        <mesh filename="package://robotiq_c2_model_visualization/meshes/robotiq_c2/collision/robotiq_85_gripper_joint_2_L.dae"/>
+        <mesh filename="package://robotiq_c2_model_visualization/meshes/collision/robotiq_85_gripper_joint_2_L.dae"/>
       </geometry>
       <origin rpy="-1.5707 1.5707 0" xyz="0 -.04843 .0127"/>
@@ -174,5 +174,5 @@
     <visual>
       <geometry>
-        <mesh filename="package://robotiq_c2_model_visualization/meshes/robotiq_c2/visual/robotiq_85_gripper_joint_2_R.dae"/>
+        <mesh filename="package://robotiq_c2_model_visualization/meshes/visual/robotiq_85_gripper_joint_2_R.dae"/>
       </geometry>
       <origin rpy="0 -1.5707 0" xyz="0 -.04843 .0127"/>
@@ -180,5 +180,5 @@
     <collision>
       <geometry>
-        <mesh filename="package://robotiq_c2_model_visualization/meshes/robotiq_c2/collision/robotiq_85_gripper_joint_2_R.dae"/>
+        <mesh filename="package://robotiq_c2_model_visualization/meshes/collision/robotiq_85_gripper_joint_2_R.dae"/>
       </geometry>
       <origin rpy="-1.5707 -1.5707 0" xyz="0 -.04843 .0127"/>
@@ -208,5 +208,5 @@
     <visual>
       <geometry>
-        <mesh filename="package://robotiq_c2_model_visualization/meshes/robotiq_c2/visual/robotiq_85_gripper_joint_3_L.dae"/>
+        <mesh filename="package://robotiq_c2_model_visualization/meshes/visual/robotiq_85_gripper_joint_3_L.dae"/>
       </geometry>
       <origin rpy="0 1.5707 0" xyz="0 -.090381 .051505"/>
@@ -214,5 +214,5 @@
     <collision>
       <geometry>
-        <mesh filename="package://robotiq_c2_model_visualization/meshes/robotiq_c2/collision/robotiq_85_gripper_joint_3_L.dae"/>
+        <mesh filename="package://robotiq_c2_model_visualization/meshes/collision/robotiq_85_gripper_joint_3_L.dae"/>
       </geometry>
       <origin rpy="-1.5707 1.5707 0" xyz="0 -.090381 .051505"/>
@@ -222,5 +222,5 @@
     <visual>
       <geometry>
-        <mesh filename="package://robotiq_c2_model_visualization/meshes/robotiq_c2/visual/robotiq_85_gripper_joint_3_R.dae"/>
+        <mesh filename="package://robotiq_c2_model_visualization/meshes/visual/robotiq_85_gripper_joint_3_R.dae"/>
       </geometry>
       <origin rpy="0 -1.5707 0" xyz="0 -.090381 .051505"/>
@@ -228,5 +228,5 @@
     <collision>
       <geometry>
-        <mesh filename="package://robotiq_c2_model_visualization/meshes/robotiq_c2/collision/robotiq_85_gripper_joint_3_R.dae"/>
+        <mesh filename="package://robotiq_c2_model_visualization/meshes/collision/robotiq_85_gripper_joint_3_R.dae"/>
       </geometry>
       <origin rpy="-1.5707 -1.5707 0" xyz="0 -.090381 .051505"/>
