Commit message: Adding fixes

File: robotiq_force_torque_sensor/urdf/robotiq_fts150.urdf.xacro (robot description, xacro)
@@ -3,5 +3,5 @@
     <xacro:macro name="robotiq_fts150" params="parent prefix *origin">
         <!-- mount the fts to the robot -->
-        <joint name="{prefix}fts_fix" type="fixed" >
+        <joint name="${prefix}fts_fix" type="fixed" >
             <!--In most cases origin would be flange adapter plate: <origin xyz="0 0 0.009" rpy="0 0 0"/> /-->
             <insert_block name="origin" />
