Commit message: Added ft

File: robotiq_force_torque_sensor/urdf/robotiq_fts300.urdf.xacro (robot description, xacro)
@@ -18,5 +18,5 @@
                 <origin xyz="0 0 0" rpy="0 0 0" />
                 <geometry>
-                    <mesh filename="package://robotiq_force_torque_sensor/meshes/visual/robotiq_fts300.stl"/>
+                    <mesh filename="package://robotiq_force_torque_sensor/meshes/visual/robotiq_fts300.dae"/>
                 </geometry>
                 <material name="black"/>
@@ -25,5 +25,5 @@
                 <origin xyz="0 0 0" rpy="0 0 0" />
                 <geometry>
-                    <mesh filename="package://robotiq_force_torque_sensor/meshes/collision/robotiq_fts300.stl"/>
+                    <mesh filename="package://robotiq_force_torque_sensor/meshes/collision/robotiq_fts300.dae"/>
                 </geometry>
             </collision>
