Commit message: fixing paths for each .dae file

File: robotiq_2f_hande_gripper_visualization/urdf/robotiq_hande_gripper.urdf.xacro (robot description, xacro)
@@ -4,5 +4,5 @@
   Author: Cristian Beltran
 -->
-  <xacro:include filename="$(find robotiq_description)/urdf/robotiq_hande_gripper.transmission.xacro" />
+  <xacro:include filename="$(find robotiq_2f_hande_gripper_visualization)/urdf/robotiq_hande_gripper.transmission.xacro" />
   <xacro:macro name="robotiq_hande_gripper" params="prefix parent *origin">
     <joint name="${prefix}robotiq_hande_base_joint" type="fixed">
@@ -20,5 +20,5 @@
         <origin rpy="0 0 0" xyz="0 0 0"/>
         <geometry>
-          <mesh filename="package://robotiq_description/meshes/hande/hand-e.dae" scale="1.0 1.0 1.0"/>
+          <mesh filename="package://robotiq_2f_hande_gripper_visualization/meshes/visual/hand-e.dae" scale="1.0 1.0 1.0"/>
         </geometry>
         <material name="Dark">
@@ -29,5 +29,5 @@
         <origin rpy="0 0 0" xyz="0 0 0"/>
         <geometry>
-          <mesh filename="package://robotiq_description/meshes/hande/hand-e-collision.dae" scale="1.0 1.0 1.0"/>
+          <mesh filename="package://robotiq_2f_hande_gripper_visualization/meshes/collision/hand-e-collision.dae" scale="1.0 1.0 1.0"/>
         </geometry>
       </collision>
@@ -42,5 +42,5 @@
         <origin rpy="0 0 0" xyz="0 0 0"/>
         <geometry>
-          <mesh filename="package://robotiq_description/meshes/hande/finger_1.dae" scale="1.0 1.0 1.0"/>
+          <mesh filename="package://robotiq_2f_hande_gripper_visualization/meshes/visual/finger_1.dae" scale="1.0 1.0 1.0"/>
         </geometry>
         <material name="DarkGray">
@@ -51,5 +51,5 @@
         <origin rpy="0 0 0" xyz="0 0 0"/>
         <geometry>
-          <mesh filename="package://robotiq_description/meshes/hande/finger_1-collision.dae" scale="1.0 1.0 1.0"/>
+          <mesh filename="package://robotiq_2f_hande_gripper_visualization/meshes/collision/finger_1-collision.dae" scale="1.0 1.0 1.0"/>
         </geometry>
       </collision>
@@ -64,5 +64,5 @@
         <origin rpy="0 0 0" xyz="0 0 0"/>
         <geometry>
-          <mesh filename="package://robotiq_description/meshes/hande/finger_2.dae" scale="1.0 1.0 1.0"/>
+          <mesh filename="package://robotiq_2f_hande_gripper_visualization/meshes/visual/finger_2.dae" scale="1.0 1.0 1.0"/>
         </geometry>
         <material name="DarkGray">
@@ -73,5 +73,5 @@
         <origin rpy="0 0 0" xyz="0 0 0"/>
         <geometry>
-          <mesh filename="package://robotiq_description/meshes/hande/finger_2-collision.dae" scale="1.0 1.0 1.0"/>
+          <mesh filename="package://robotiq_2f_hande_gripper_visualization/meshes/collision/finger_2-collision.dae" scale="1.0 1.0 1.0"/>
         </geometry>
       </collision>
